File: Comm.brd (EAGLE design)
At the start: 30 x 60 mm, 36 parts, among them SW1 THAU13-AB-R, SW2 THAU13-AB-R, SW3 TVAF06-A020B-R, SW4 TVAF06-A020B-R, U4 OPA340N, U5 DRIVER-LV8548MC-AH(SOIC10), U6 I-02247_NJM2845

Commit message: fix register value
Parts:
- R10: value (none) -> 47k
- R11: value (none) -> 10k
- R12: value (none) -> 22k
- R13: value (none) -> 5.1k
- R2: value 200k -> 220k
- R4: value 1k -> 10k
- R7: value 100k -> 0
- R8: value 100k -> 47k
- R9: value (none) -> 82k
Changed lines of the file:
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@@
 <grid distance="50" unitdist="mil" unit="mm" style="dots" multiple="1" display="yes" altdistance="5" altunitdist="mil" altunit="mm"/>
 <layers>
-<layer number="1" name="Top" color="4" fill="1" visible="yes" active="yes"/>
+<layer number="1" name="Top" color="4" fill="1" visible="no" active="yes"/>
 <layer number="2" name="Route2" color="16" fill="1" visible="no" active="no"/>
 <layer number="3" name="Route3" color="17" fill="1" visible="no" active="no"/>
@@
 <layer number="19" name="Unrouted" color="6" fill="1" visible="yes" active="yes"/>
 <layer number="20" name="Dimension" color="24" fill="1" visible="yes" active="yes"/>
-<layer number="21" name="tPlace" color="7" fill="1" visible="yes" active="yes"/>
+<layer number="21" name="tPlace" color="7" fill="1" visible="no" active="yes"/>
 <layer number="22" name="bPlace" color="7" fill="1" visible="yes" active="yes"/>
-<layer number="23" name="tOrigins" color="15" fill="1" visible="yes" active="yes"/>
+<layer number="23" name="tOrigins" color="15" fill="1" visible="no" active="yes"/>
 <layer number="24" name="bOrigins" color="15" fill="1" visible="yes" active="yes"/>
-<layer number="25" name="tNames" color="7" fill="1" visible="yes" active="yes"/>
+<layer number="25" name="tNames" color="7" fill="1" visible="no" active="yes"/>
 <layer number="26" name="bNames" color="7" fill="1" visible="yes" active="yes"/>
 <layer number="27" name="tValues" color="7" fill="1" visible="no" active="yes"/>
 <layer number="28" name="bValues" color="7" fill="1" visible="no" active="yes"/>
-<layer number="29" name="tStop" color="7" fill="3" visible="yes" active="yes"/>
+<layer number="29" name="tStop" color="7" fill="3" visible="no" active="yes"/>
 <layer number="30" name="bStop" color="7" fill="6" visible="no" active="yes"/>
 <layer number="31" name="tCream" color="7" fill="4" visible="no" active="yes"/>
@@
 <layer number="37" name="tTest" color="7" fill="1" visible="no" active="yes"/>
 <layer number="38" name="bTest" color="7" fill="1" visible="no" active="yes"/>
-<layer number="39" name="tKeepout" color="4" fill="11" visible="yes" active="yes"/>
+<layer number="39" name="tKeepout" color="4" fill="11" visible="no" active="yes"/>
 <layer number="40" name="bKeepout" color="1" fill="11" visible="yes" active="yes"/>
-<layer number="41" name="tRestrict" color="4" fill="10" visible="yes" active="yes"/>
+<layer number="41" name="tRestrict" color="4" fill="10" visible="no" active="yes"/>
 <layer number="42" name="bRestrict" color="1" fill="10" visible="yes" active="yes"/>
 <layer number="43" name="vRestrict" color="2" fill="10" visible="no" active="yes"/>
@@
 <layer number="49" name="Reference" color="7" fill="1" visible="no" active="yes"/>
 <layer number="50" name="dxf" color="7" fill="1" visible="no" active="no"/>
-<layer number="51" name="tDocu" color="7" fill="1" visible="yes" active="yes"/>
+<layer number="51" name="tDocu" color="7" fill="1" visible="no" active="yes"/>
 <layer number="52" name="bDocu" color="7" fill="1" visible="yes" active="yes"/>
 <layer number="53" name="tGND_GNDA" color="7" fill="1" visible="no" active="no"/>
@@
 <attribute name="VALUE" x="-5.715" y="-5.715" size="1.27" layer="28" rot="MR0"/>
 </element>
-<element name="R8" library="rcl" library_urn="urn:adsk.eagle:library:334" package="R0603" package3d_urn="urn:adsk.eagle:package:23555/3" value="100k" x="-6.35" y="-6.35" smashed="yes" rot="MR180">
+<element name="R8" library="rcl" library_urn="urn:adsk.eagle:library:334" package="R0603" package3d_urn="urn:adsk.eagle:package:23555/3" value="47k" x="-6.35" y="-6.35" smashed="yes" rot="MR180">
 <attribute name="NAME" x="-3.937" y="-6.35" size="1.016" layer="26" font="vector" rot="MR180" align="center"/>
 <attribute name="POPULARITY" value="77" x="-6.35" y="-6.35" size="1.778" layer="28" rot="MR180" display="off"/>
@@
 <attribute name="VALUE" x="-6.985" y="-4.445" size="1.27" layer="28" rot="MR180"/>
 </element>
-<element name="R4" library="rcl" library_urn="urn:adsk.eagle:library:334" package="R0603" package3d_urn="urn:adsk.eagle:package:23555/3" value="1k" x="-6.35" y="-19.05" smashed="yes" rot="MR0">
+<element name="R4" library="rcl" library_urn="urn:adsk.eagle:library:334" package="R0603" package3d_urn="urn:adsk.eagle:package:23555/3" value="10k" x="-6.35" y="-19.05" smashed="yes" rot="MR0">
 <attribute name="NAME" x="-8.89" y="-19.05" size="1.016" layer="26" font="vector" rot="MR0" align="center"/>
 <attribute name="POPULARITY" value="77" x="-6.35" y="-19.05" size="1.778" layer="28" rot="MR0" display="off"/>
@@
 <attribute name="VALUE" x="-5.715" y="-20.955" size="1.27" layer="28" rot="MR0"/>
 </element>
-<element name="R7" library="rcl" library_urn="urn:adsk.eagle:library:334" package="R0603" package3d_urn="urn:adsk.eagle:package:23555/3" value="100k" x="-6.35" y="-16.51" smashed="yes" rot="MR0">
+<element name="R7" library="rcl" library_urn="urn:adsk.eagle:library:334" package="R0603" package3d_urn="urn:adsk.eagle:package:23555/3" value="0" x="-6.35" y="-16.51" smashed="yes" rot="MR0">
 <attribute name="NAME" x="-8.89" y="-16.51" size="1.016" layer="26" font="vector" rot="MR0" align="center"/>
 <attribute name="POPULARITY" value="77" x="-6.35" y="-16.51" size="1.778" layer="28" rot="MR0" display="off"/>
@@
 <attribute name="VALUE" x="0.635" y="-23.495" size="1.27" layer="28" rot="MR0"/>
 </element>
-<element name="R2" library="rcl" library_urn="urn:adsk.eagle:library:334" package="R0603" package3d_urn="urn:adsk.eagle:package:23555/3" value="200k" x="6.35" y="-6.35" smashed="yes" rot="MR0">
+<element name="R2" library="rcl" library_urn="urn:adsk.eagle:library:334" package="R0603" package3d_urn="urn:adsk.eagle:package:23555/3" value="220k" x="6.35" y="-6.35" smashed="yes" rot="MR0">
 <attribute name="NAME" x="4.064" y="-6.35" size="1.016" layer="26" font="vector" rot="MR0" align="center"/>
 <attribute name="POPULARITY" value="77" x="6.35" y="-6.35" size="1.778" layer="28" rot="MR0" display="off"/>
@@
 <attribute name="VALUE" x="10.16" y="8.255" size="0.8128" layer="27" font="vector" rot="R180"/>
 </element>
-<element name="R9" library="rcl" library_urn="urn:adsk.eagle:library:334" package="R0603" package3d_urn="urn:adsk.eagle:package:23555/3" value="" x="12.065" y="-15.24" smashed="yes" rot="MR270">
+<element name="R9" library="rcl" library_urn="urn:adsk.eagle:library:334" package="R0603" package3d_urn="urn:adsk.eagle:package:23555/3" value="82k" x="12.065" y="-15.24" smashed="yes" rot="MR270">
 <attribute name="NAME" x="10.668" y="-15.24" size="1.016" layer="26" font="vector" rot="MR270" align="center"/>
 <attribute name="POPULARITY" value="77" x="12.065" y="-15.24" size="1.778" layer="28" rot="MR270" display="off"/>
@@
 <attribute name="VALUE" x="13.97" y="-14.605" size="1.27" layer="28" rot="MR270"/>
 </element>
-<element name="R10" library="rcl" library_urn="urn:adsk.eagle:library:334" package="R0603" package3d_urn="urn:adsk.eagle:package:23555/3" value="" x="9.525" y="-12.7" smashed="yes" rot="MR270">
+<element name="R10" library="rcl" library_urn="urn:adsk.eagle:library:334" package="R0603" package3d_urn="urn:adsk.eagle:package:23555/3" value="47k" x="9.525" y="-12.7" smashed="yes" rot="MR270">
 <attribute name="NAME" x="8.255" y="-12.7" size="1.016" layer="26" font="vector" rot="MR270" align="center"/>
 <attribute name="POPULARITY" value="77" x="9.525" y="-12.7" size="1.778" layer="28" rot="MR270" display="off"/>
@@
 <attribute name="VALUE" x="11.43" y="-12.065" size="1.27" layer="28" rot="MR270"/>
 </element>
-<element name="R11" library="rcl" library_urn="urn:adsk.eagle:library:334" package="R0603" package3d_urn="urn:adsk.eagle:package:23555/3" value="" x="9.525" y="-8.89" smashed="yes" rot="MR270">
+<element name="R11" library="rcl" library_urn="urn:adsk.eagle:library:334" package="R0603" package3d_urn="urn:adsk.eagle:package:23555/3" value="10k" x="9.525" y="-8.89" smashed="yes" rot="MR270">
 <attribute name="NAME" x="8.382" y="-8.89" size="1.016" layer="26" font="vector" rot="MR270" align="center"/>
 <attribute name="POPULARITY" value="77" x="9.525" y="-8.89" size="1.778" layer="28" rot="MR270" display="off"/>
@@
 <attribute name="VALUE" x="11.43" y="-8.255" size="1.27" layer="28" rot="MR270"/>
 </element>
-<element name="R12" library="rcl" library_urn="urn:adsk.eagle:library:334" package="R0603" package3d_urn="urn:adsk.eagle:package:23555/3" value="" x="-9.525" y="-12.7" smashed="yes" rot="MR270">
+<element name="R12" library="rcl" library_urn="urn:adsk.eagle:library:334" package="R0603" package3d_urn="urn:adsk.eagle:package:23555/3" value="22k" x="-9.525" y="-12.7" smashed="yes" rot="MR270">
 <attribute name="NAME" x="-10.795" y="-15.113" size="1.016" layer="26" font="vector" rot="MR270" align="center"/>
 <attribute name="POPULARITY" value="77" x="-9.525" y="-12.7" size="1.778" layer="28" rot="MR270" display="off"/>
@@
 <attribute name="VALUE" x="-7.62" y="-12.065" size="1.27" layer="28" rot="MR270"/>
 </element>
-<element name="R13" library="rcl" library_urn="urn:adsk.eagle:library:334" package="R0603" package3d_urn="urn:adsk.eagle:package:23555/3" value="" x="-9.525" y="-8.89" smashed="yes" rot="MR270">
+<element name="R13" library="rcl" library_urn="urn:adsk.eagle:library:334" package="R0603" package3d_urn="urn:adsk.eagle:package:23555/3" value="5.1k" x="-9.525" y="-8.89" smashed="yes" rot="MR270">
 <attribute name="NAME" x="-8.382" y="-8.89" size="1.016" layer="26" font="vector" rot="MR270" align="center"/>
 <attribute name="POPULARITY" value="77" x="-9.525" y="-8.89" size="1.778" layer="28" rot="MR270" display="off"/>
